Commit message: - Fixed tf link for lidar and base_link - Corrected the position of footprint_link - Added a plugin package to publish 3D Bounding Box of a model from Gazebo to ROS 2 - Configured the correct TF tree structure: world -> odom -> base_link - Implemented tf_odom_broadcaster node to handle the base_link to odom transform - Added odom.rviz configuration file for RViz2 visualization - Integrated complete ground truth positioning by extracting the pose from Gazebo using the p3d plugin

File: air_description/urdf/bases/sd_twizy_body.urdf.xacro (robot description, xacro)
@@ -29,5 +29,5 @@
     <parent link="base_link"/>
     <child link="footprint_link"/>
-    <origin xyz="${wheelbase} 0 ${clearance}" rpy="0 0 0"/>
+    <origin xyz="0 0 ${-clearance}" rpy="0 0 0"/>
   </joint>
     <joint name="chassis_joint" type="fixed">
@@ -49,5 +49,4 @@
         <geometry>
           <mesh filename="file:///$(find air_description)/meshes/SDTwizy.stl" scale="0.01 0.01 0.01"/>
-          <!-- <mesh filename="file:///$(find air_description)/models/twizy/meshes/SDTwizy.stl" scale="0.01 0.01 0.01"/> -->
         </geometry>
         <material name="chassis_color" />
@@ -57,5 +56,4 @@
         <geometry>
           <mesh filename="file:///$(find air_description)/meshes/SDTwizy_collision.stl" scale="0.01 0.01 0.01"/>
-          <!-- <mesh filename="file:///$(find air_description)/models/twizy/meshes/SDTwizy_collision.stl" scale="0.01 0.01 0.01"/> -->
         </geometry>
       </collision>

File: air_description/urdf/sd_twizy.urdf.xacro (robot description, xacro)
@@ -30,5 +30,5 @@
   <xacro:include filename="$(find velodyne_description)/urdf/VLP-16.urdf.xacro"/>
   <xacro:VLP-16 parent="base_link" name="velodyne" topic="/velodyne_points" organize_cloud="${organize_cloud}" hz="5" samples="440" gpu="${gpu}">
-    <origin xyz="-0.681 0 1.445" rpy="0 -${1.5*M_PI/180.0} 0"/>
+    <origin xyz="0 0 1.445" rpy="0 -${1.5*M_PI/180.0} 0"/>
   </xacro:VLP-16>
   <xacro:blackfly_camera frlr_prefix="front" lrc_prefix="left">
@@ -58,9 +58,8 @@
   <gazebo>
     <plugin name="libgazebo_ros_p3d" filename="libgazebo_ros_p3d.so">
-      <ros>
-          <namespace>p3d</namespace>
+       <ros>
           <remapping>odom:=base_pose_ground_truth</remapping>
         </ros>
-          <frame_name>map</frame_name>
+          <frame_name>world</frame_name>
           <body_name>base_link</body_name>
           <update_rate>200.0</update_rate>
@@ -95,3 +94,9 @@
     </plugin>
   </gazebo>
+  <gazebo>
+    <plugin name="bounding_box_plugin" filename="/root/ros2_ws/install/bounding_box_plugin/lib/bounding_box_plugin/libbounding_box_plugin.so">
+      <update_rate>5.0</update_rate>
+      <frame_id>world</frame_id>
+    </plugin>
+  </gazebo>
 </robot>
